File: pcb/controller/controller.kicad_sch (KiCad schematic)
At the start: 37 parts, among them J1 JST-HX_01x03, J2 Barrel_Jack, U1 Teensy4.0

Commit message: Widgetpad controller v0.2
Connections:
- net +3V3: now also U1.31 (3V3)
- no-connect marks 27 -> 26
Changed lines of the file:
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@@
   (no_connect (at 100.33 82.55))
   (no_connect (at 100.33 85.09))
-  (no_connect (at 100.33 100.33))
   (no_connect (at 100.33 102.87))
   (wire (pts (xy 25.4 41.91) (xy 44.45 41.91))
@@
     (stroke (width 0) (type solid) (color 0 0 0 0))
   )
-  (wire (pts (xy 100.33 97.79) (xy 114.3 97.79))
+  (wire (pts (xy 100.33 97.79) (xy 105.41 97.79))
+    (stroke (width 0) (type solid) (color 0 0 0 0))
+  )
+  (wire (pts (xy 100.33 100.33) (xy 116.84 100.33))
     (stroke (width 0) (type solid) (color 0 0 0 0))
   )
@@
     (stroke (width 0) (type solid) (color 0 0 0 0))
   )
+  (wire (pts (xy 105.41 88.9) (xy 110.49 88.9))
+    (stroke (width 0) (type solid) (color 0 0 0 0))
+  )
+  (wire (pts (xy 105.41 97.79) (xy 105.41 88.9))
+    (stroke (width 0) (type solid) (color 0 0 0 0))
+  )
+  (wire (pts (xy 110.49 88.9) (xy 110.49 91.44))
+    (stroke (width 0) (type solid) (color 0 0 0 0))
+  )
   (wire (pts (xy 110.49 105.41) (xy 100.33 105.41))
     (stroke (width 0) (type solid) (color 0 0 0 0))
   )
-  (wire (pts (xy 114.3 97.79) (xy 114.3 100.33))
+  (wire (pts (xy 116.84 97.79) (xy 116.84 100.33))
     (stroke (width 0) (type solid) (color 0 0 0 0))
   )
@@
     (pin "1")
   )
+  (symbol (lib_id "power:+3V3") (at 116.84 97.79 0) (unit 1)
+    (in_bom yes) (on_board yes)
+    (property "Reference" "#PWR?" (id 0) (at 116.84 101.6 0)
+      (effects (font (size 1.27 1.27)) hide)
+    )
+    (property "Value" "+3V3" (id 1) (at 117.221 93.3958 0))
+    (property "Footprint" "" (id 2) (at 116.84 97.79 0)
+      (effects (font (size 1.27 1.27)) hide)
+    )
+    (property "Datasheet" "" (id 3) (at 116.84 97.79 0)
+      (effects (font (size 1.27 1.27)) hide)
+    )
+    (pin "1")
+  )
   (symbol (lib_id "power:+3V3") (at 151.13 17.78 90) (unit 1)
     (in_bom yes) (on_board yes)
@@
     (pin "1")
   )
-  (symbol (lib_id "power:GND") (at 114.3 100.33 0) (unit 1)
-    (in_bom yes) (on_board yes)
-    (property "Reference" "#PWR03" (id 0) (at 114.3 106.68 0)
-      (effects (font (size 1.27 1.27)) hide)
-    )
-    (property "Value" "GND" (id 1) (at 114.427 104.7242 0))
-    (property "Footprint" "" (id 2) (at 114.3 100.33 0)
-      (effects (font (size 1.27 1.27)) hide)
-    )
-    (property "Datasheet" "" (id 3) (at 114.3 100.33 0)
+  (symbol (lib_id "power:GND") (at 110.49 91.44 0) (unit 1)
+    (in_bom yes) (on_board yes)
+    (property "Reference" "#PWR03" (id 0) (at 110.49 97.79 0)
+      (effects (font (size 1.27 1.27)) hide)
+    )
+    (property "Value" "GND" (id 1) (at 110.617 95.8342 0))
+    (property "Footprint" "" (id 2) (at 110.49 91.44 0)
+      (effects (font (size 1.27 1.27)) hide)
+    )
+    (property "Datasheet" "" (id 3) (at 110.49 91.44 0)
       (effects (font (size 1.27 1.27)) hide)
     )
@@
       (reference "#PWR036") (unit 1) (value "+5V") (footprint "")
     )
+    (path "/1cd6677e-ecaf-469b-a05b-b62c3786ebae"
+      (reference "#PWR?") (unit 1) (value "+3V3") (footprint "")
+    )
     (path "/00000000-0000-0000-0000-000061a093c3"
